File: vhf_uhf_IQ_Modulator.sch (KiCad schematic (older format))
At the start: 75 parts

Commit message: a/d
Parts:
- added U? (x2): MCP3421A0T-E/CH, symbol MCP3421A0T-E/CH
- added U?: MCP4728, Housings_SSOP:MSOP-10_3x3mm_Pitch0.5mm, symbol MCP4728
- U?: value orange_pi_zero -> Orange Pi zero
Connections:
- net PDet: now also U?.1 (Vin+)
- net SDA: now also U?.103 (TWI0_SDA_/_PA12), U?.7 (SDA)
- net PowerDown: now reaches U?.7 (PWD)
- net OCX_EN: now reaches U?.2 (OE)
- net SLC: now reaches U?.105 (TWI0_SCK_/_PA11), U?.8 (SCL)
- net PA_ON: now reaches U?.10 (Pow_Down)
- new net VBat: U?.1 (Vin+)
Other:
- moved on the sheet: C?, L?
Changed lines of the file:
@@
 P 4700 4600
 F 0 "U?" H 4800 5600 60  0000 C CNN
-F 1 "orange_pi_zero" H 4850 2950 60  0000 C CNN
+F 1 "Orange Pi zero" H 4600 3000 60  0000 C CNN
 F 2 "" H 4450 5400 60  0000 C CNN
 F 3 "" H 4450 5400 60  0000 C CNN
@@
 Connection ~ 8550 2800
 Wire Wire Line
-	6400 4050 6100 4050
-Wire Wire Line
 	6100 4050 6100 3600
 Wire Wire Line
@@
 L L L?
 U 1 1 5A2373B0
-P 12850 1800
-F 0 "L?" V 12800 1800 50  0000 C CNN
-F 1 "L" V 12925 1800 50  0000 C CNN
-F 2 "" H 12850 1800 50  0001 C CNN
-F 3 "" H 12850 1800 50  0001 C CNN
-	1    12850 1800
+P 12850 1550
+F 0 "L?" V 12800 1550 50  0000 C CNN
+F 1 "L" V 12925 1550 50  0000 C CNN
+F 2 "" H 12850 1550 50  0001 C CNN
+F 3 "" H 12850 1550 50  0001 C CNN
+	1    12850 1550
 	1    0    0    -1
 $EndComp
@@
 L C_Small C?
 U 1 1 5A2374AB
-P 13200 2050
-F 0 "C?" H 13210 2120 50  0000 L CNN
-F 1 "C_Small" H 13210 1970 50  0000 L CNN
-F 2 "" H 13200 2050 50  0001 C CNN
-F 3 "" H 13200 2050 50  0001 C CNN
-	1    13200 2050
+P 13200 1800
+F 0 "C?" H 13210 1870 50  0000 L CNN
+F 1 "C_Small" H 13210 1720 50  0000 L CNN
+F 2 "" H 13200 1800 50  0001 C CNN
+F 3 "" H 13200 1800 50  0001 C CNN
+	1    13200 1800
 	-1   0    0    1
 $EndComp
@@
 L C_Small C?
 U 1 1 5A237595
-P 13150 1600
-F 0 "C?" H 13160 1670 50  0000 L CNN
-F 1 "C_Small" H 13160 1520 50  0000 L CNN
-F 2 "" H 13150 1600 50  0001 C CNN
-F 3 "" H 13150 1600 50  0001 C CNN
-	1    13150 1600
+P 13150 1350
+F 0 "C?" H 13160 1420 50  0000 L CNN
+F 1 "C_Small" H 13160 1270 50  0000 L CNN
+F 2 "" H 13150 1350 50  0001 C CNN
+F 3 "" H 13150 1350 50  0001 C CNN
+	1    13150 1350
 	-1   0    0    1
 $EndComp
 Wire Wire Line
-	12850 2250 12850 1950
-Wire Wire Line
-	12850 1950 13200 1950
+	12850 1700 13200 1700
 $Comp
 L GND #PWR?
 U 1 1 5A237928
-P 13200 2200
-F 0 "#PWR?" H 13200 1950 50  0001 C CNN
-F 1 "GND" H 13200 2050 50  0000 C CNN
-F 2 "" H 13200 2200 50  0001 C CNN
-F 3 "" H 13200 2200 50  0001 C CNN
-	1    13200 2200
+P 13200 2000
+F 0 "#PWR?" H 13200 1750 50  0001 C CNN
+F 1 "GND" H 13200 1850 50  0000 C CNN
+F 2 "" H 13200 2000 50  0001 C CNN
+F 3 "" H 13200 2000 50  0001 C CNN
+	1    13200 2000
 	1    0    0    -1
 $EndComp
@@
 L GND #PWR?
 U 1 1 5A237A2F
-P 13150 1750
-F 0 "#PWR?" H 13150 1500 50  0001 C CNN
-F 1 "GND" H 13150 1600 50  0000 C CNN
-F 2 "" H 13150 1750 50  0001 C CNN
-F 3 "" H 13150 1750 50  0001 C CNN
-	1    13150 1750
+P 13150 1500
+F 0 "#PWR?" H 13150 1250 50  0001 C CNN
+F 1 "GND" H 13150 1350 50  0000 C CNN
+F 2 "" H 13150 1500 50  0001 C CNN
+F 3 "" H 13150 1500 50  0001 C CNN
+	1    13150 1500
 	1    0    0    -1
 $EndComp
@@
 L +5V #PWR?
 U 1 1 5A237AF7
-P 12850 1450
-F 0 "#PWR?" H 12850 1300 50  0001 C CNN
-F 1 "+5V" H 12850 1590 50  0000 C CNN
-F 2 "" H 12850 1450 50  0001 C CNN
-F 3 "" H 12850 1450 50  0001 C CNN
-	1    12850 1450
-	1    0    0    -1
-$EndComp
-Wire Wire Line
-	12850 1450 12850 1650
-Wire Wire Line
-	13150 1500 12850 1500
-Connection ~ 12850 1500
-Wire Wire Line
-	13150 1700 13150 1750
-Wire Wire Line
-	13200 2150 13200 2200
+P 12850 1200
+F 0 "#PWR?" H 12850 1050 50  0001 C CNN
+F 1 "+5V" H 12850 1340 50  0000 C CNN
+F 2 "" H 12850 1200 50  0001 C CNN
+F 3 "" H 12850 1200 50  0001 C CNN
+	1    12850 1200
+	1    0    0    -1
+$EndComp
+Wire Wire Line
+	12850 1200 12850 1400
+Wire Wire Line
+	13150 1250 12850 1250
+Connection ~ 12850 1250
+Wire Wire Line
+	13150 1450 13150 1500
 $Comp
 L C_Small C?
@@
 Wire Wire Line
 	6250 6750 6550 6750
-Text Label 6550 6750 0    60   ~ 0
-SCL
 Wire Wire Line
 	6250 6850 6550 6850
-Text Label 6550 6850 0    60   ~ 0
-SDA
 $Comp
 L R R?
@@
 Text Label 6300 7150 0    60   ~ 0
 INT
+$Comp
+L MCP3421A0T-E/CH U?
+U 1 1 5A83B056
+P 9600 6900
+F 0 "U?" H 9200 7200 50  0000 L CNN
+F 1 "MCP3421A0T-E/CH" H 9700 7200 50  0000 L CNN
+F 2 "" H 9600 6900 50  0001 C CIN
+F 3 "" H 9600 6900 50  0001 C CNN
+	1    9600 6900
+	-1   0    0    1
+$EndComp
+$Comp
+L MCP3421A0T-E/CH U?
+U 1 1 5A83DF17
+P 9600 8050
+F 0 "U?" H 9200 8350 50  0000 L CNN
+F 1 "MCP3421A0T-E/CH" H 9700 8350 50  0000 L CNN
+F 2 "" H 9600 8050 50  0001 C CIN
+F 3 "" H 9600 8050 50  0001 C CNN
+	1    9600 8050
+	-1   0    0    1
+$EndComp
+$Comp
+L MCP4728 U?
+U 1 1 5A83EBAC
+P 7250 2400
+F 0 "U?" H 6750 2650 50  0000 L CNN
+F 1 "MCP4728" H 7750 2650 50  0000 R CNN
+F 2 "Housings_SSOP:MSOP-10_3x3mm_Pitch0.5mm" H 7250 1800 50  0001 C CNN
+F 3 "" H 7250 2650 50  0001 C CNN
+	1    7250 2400
+	1    0    0    -1
+$EndComp
+Text GLabel 10300 7000 2    60   Input ~ 0
+PDet
+Wire Wire Line
+	10100 7000 10300 7000
+Text GLabel 6550 6850 2    60   Input ~ 0
+SDA
+Text GLabel 6550 6750 2    60   Input ~ 0
+SCL
+Wire Wire Line
+	6100 4050 6350 4050
+Text GLabel 6100 3800 2    60   Input ~ 0
+SDA
+Text GLabel 6250 4150 3    60   Input ~ 0
+SLC
+Wire Wire Line
+	6350 3850 6350 3300
+Text GLabel 6350 3300 2    60   Input ~ 0
+OCX_EN
+Wire Wire Line
+	10100 8150 10350 8150
+Text GLabel 10350 8150 2    60   Input ~ 0
+VBat
+Text GLabel 12950 2250 1    60   Input ~ 0
+PA_ON
+Wire Wire Line
+	13200 1900 13200 2000
+Wire Wire Line
+	12850 1700 12850 2250
+Wire Wire Line
+	9750 3250 9750 4200
+Text GLabel 9750 4200 3    60   Input ~ 0
+PowerDown
 $EndSCHEMATC

Commit message: 2m filter and rf switch
Parts:
- removed C? (x2): C_Small, symbol C_Small
- removed F?: LFCN-80, symbol LFCN-80
- removed U?: HMC544A, symbol HMC544A
- removed U?: 74AHC1G04, symbol 74AHC1G04
- removed U?: MCP3421A0T-E/CH, symbol MCP3421A0T-E/CH
- removed U?: MCP4728, Housings_SSOP:MSOP-10_3x3mm_Pitch0.5mm, symbol MCP4728
- added C? (x3): C_Small, symbol C_Small
- added J?: Conn_01x03, symbol Conn_01x03
- added L? (x4): L, symbol L
- added R? (x3): R, symbol R
- U?: symbol MCP3421A0T-E/CH -> MCP3421A0T-E/CH-RESCUE-vhf_uhf_IQ_Modulator
Connections:
- net GND: now also C?.1, C?.1, C?.1, R?.1
- net at R?.2: now also L?.1
- net at U?.2 (RF_In): now also J?.1 (Pin_1)
- net at C?.1: now also J?.2 (Pin_2)
- new net: J?.3 (Pin_3), R?.2
- new net: C?.2, L?.1, L?.2 (x3)
- new net: L?.2, R?.1
- new net: R?.1, R?.2, R?.2
Other:
- note added: "Check connection\n"
- note removed: "2m BPF"
- note removed: "RF Switch 70cm/2m"
- moved on the sheet: U?
