File: vhf_uhf_IQ_Modulator.kicad_pcb (KiCad board)
At the start: 2 copper layers, 2 parts

Commit message: Created Bom and pcbedge
Parts:
- removed REF**: orange pi zero, orangepi-zero:orange pi zero
- removed REF**: orange pi zero, orangepi-zero:orangepi-zero
- added BT1: 3.3V Battery_Cell, Battery_Holders:Keystone_103_1x20mm-CoinCell, F.Cu at (109.2, 67.3)
- added C1: 1uF 16V, Capacitors_Tantalum_SMD:CP_Tantalum_Case-R_EIA-2012-12_Reflow, F.Cu at (174.6, 58.4)
- added C10: 4.7uF 16V, Capacitors_SMD:C_0805_HandSoldering, F.Cu at (175.3, 97.8)
- added C11: 2200pF, Capacitors_SMD:C_0805_HandSoldering, F.Cu at (168.9, 92.7)
- added C12: 2200pF, Capacitors_SMD:C_0805_HandSoldering, F.Cu at (175.9, 88.3)
- added C13: 1uF 16V, Capacitors_Tantalum_SMD:CP_Tantalum_Case-R_EIA-2012-12_Reflow, F.Cu at (175.3, 91.4)
- added C14: 1nF, Capacitors_SMD:C_0805_HandSoldering, F.Cu at (168.9, 97.8)
- added C15: 1uF 16V, Capacitors_Tantalum_SMD:CP_Tantalum_Case-R_EIA-2012-12_Reflow, F.Cu at (162.6, 102.9)
- added C16: 100pF, Capacitors_SMD:C_0805_HandSoldering, F.Cu at (158.8, 97.8)
- added C17: 1uF 16V, Capacitors_Tantalum_SMD:CP_Tantalum_Case-R_EIA-2012-12_Reflow, F.Cu at (170.2, 83.8)
- added C18: 27pF, Capacitors_SMD:C_0805_HandSoldering, F.Cu at (184.2, 90.2)
- added C19: 220pF, Capacitors_SMD:C_0805_HandSoldering, F.Cu at (176.5, 86.4)
- added C2: 1uF 16V, Capacitors_Tantalum_SMD:CP_Tantalum_Case-R_EIA-2012-12_Reflow, F.Cu at (159.4, 85.1)
- added C20: 1uF 16V, Capacitors_Tantalum_SMD:CP_Tantalum_Case-R_EIA-2012-12_Reflow, F.Cu at (163.8, 97.8)
- added C21: 100pF, Capacitors_SMD:C_0805_HandSoldering, F.Cu at (154.9, 82.5)
- added C22: 33pF, Capacitors_SMD:C_0805_HandSoldering, F.Cu at (157.5, 101.6)
- added C23: 10uF 16V, Capacitors_SMD:C_0805_HandSoldering, F.Cu at (168.9, 101.6)
- added C24: 15pF, Capacitors_SMD:C_0805_HandSoldering, F.Cu at (153.7, 97.8)
- added C25: 10uF 16V, Capacitors_SMD:C_0805_HandSoldering, F.Cu at (182.9, 99.1)
- added C26: 100nF, Capacitors_SMD:C_0805_HandSoldering, F.Cu at (182.9, 87.6)
- added C27: 10uF 16V, Capacitors_SMD:C_0805_HandSoldering, F.Cu at (182.9, 95.2)
- added C28: 220pF, Capacitors_SMD:C_0805_HandSoldering, F.Cu at (163.8, 87.6)
- added C29: 33pF, Capacitors_SMD:C_0805_HandSoldering, F.Cu at (153.7, 87.6)
- added C3: 1uF 16V, Capacitors_Tantalum_SMD:CP_Tantalum_Case-R_EIA-2012-12_Reflow, F.Cu at (161.9, 58.4)
- added C30: 33pF, Capacitors_SMD:C_0805_HandSoldering, F.Cu at (163.8, 82.5)
- added C31: 33pF, Capacitors_SMD:C_0805_HandSoldering, F.Cu at (163.8, 92.7)
- added C32: 100nF, Capacitors_SMD:C_0805_HandSoldering, F.Cu at (175.3, 83.8)
- added C33: 22pF, Capacitors_SMD:C_0805_HandSoldering, F.Cu at (180.3, 83.8)
- added C4: 3.3pF, Capacitors_SMD:C_0805_HandSoldering, F.Cu at (158.8, 92.7)
- added C5: 10uF 16V, Capacitors_SMD:C_0805_HandSoldering, F.Cu at (181.6, 63.5)
- added C6: 2200pF, Capacitors_SMD:C_0805_HandSoldering, F.Cu at (154.3, 85.1)
- added C7: 2200pF, Capacitors_SMD:C_0805_HandSoldering, F.Cu at (168.9, 88.9)
- added C8: 10uF 16V, Capacitors_SMD:C_0805_HandSoldering, F.Cu at (158.8, 82.5)
- added C9: 1nF, Capacitors_SMD:C_0805_HandSoldering, F.Cu at (158.8, 87.6)
- added D1: 1N4148, Diodes_SMD:D_SOD-123, F.Cu at (153.7, 92.7)
- added J1: Conn_01x06, Connectors_Molex:Molex_KK-6410-06_06x2.54mm_Straight, F.Cu at (142.2, 78.7)
- added J2: TEST_1P, Inductors_SMD:L_0805_HandSoldering, F.Cu at (184.2, 92.7)
- added J3: Audio-Jack-3, Connectors_Molex:Molex_KK-6410-03_03x2.54mm_Straight, F.Cu at (158.8, 113.0)
- added J4: CONN_01X04, Connectors_Molex:Molex_KK-6410-04_04x2.54mm_Straight, F.Cu at (199.4, 80.0)
- added J5: SMA Edge FM, Connectors_Molex:Molex_SMA_Jack_Edge_Mount, F.Cu at (179.1, 104.1)
- added L1: 33nF, Capacitors_SMD:C_0805_HandSoldering, F.Cu at (188.0, 99.1)
- added L2: 33nH, Inductors_SMD:L_0805_HandSoldering, F.Cu at (161.3, 80.0)
- added L3: 22nF, Capacitors_SMD:C_0805_HandSoldering, F.Cu at (175.3, 94.0)
- added L4: 33nH, Inductors_SMD:L_0805_HandSoldering, F.Cu at (154.9, 77.5)
- added L5: 33nF, Capacitors_SMD:C_0805_HandSoldering, F.Cu at (185.4, 83.8)
- added L6: 56nH, Inductors_SMD:L_0805_HandSoldering, F.Cu at (154.9, 73.7)
- added L7: 110nH, Inductors_SMD:L_0805_HandSoldering, F.Cu at (177.8, 80.0)
- added L8: 110nH, Inductors_SMD:L_0805_HandSoldering, F.Cu at (179.1, 73.7)
- added L9: 56nH, Inductors_SMD:L_0805_HandSoldering, F.Cu at (154.9, 80.0)
- added Q1: BC817-40, TO_SOT_Packages_SMD:SOT-23, F.Cu at (186.7, 72.4)
- added Q2: BC817-40, TO_SOT_Packages_SMD:SOT-23, F.Cu at (186.7, 76.2)
- added Q3: BC817-40, TO_SOT_Packages_SMD:SOT-23, F.Cu at (182.9, 76.2)
- added R1: 10k, Resistors_SMD:R_0805_HandSoldering, F.Cu at (166.4, 80.0)
- added R10: 2k2, Resistors_SMD:R_0805_HandSoldering, F.Cu at (165.1, 73.7)
- added R11: OC, Resistors_SMD:R_0805_HandSoldering, F.Cu at (154.9, 68.6)
- added R12: 0, Resistors_SMD:R_0805_HandSoldering, F.Cu at (165.1, 66.0)
- added R13: 0, Resistors_SMD:R_0805_HandSoldering, F.Cu at (160.0, 71.1)
- added R14: 10k, Resistors_SMD:R_0805_HandSoldering, F.Cu at (160.0, 63.5)
- added R15: 0, Resistors_SMD:R_0805_HandSoldering, F.Cu at (160.0, 66.0)
- added R16: OC, Resistors_SMD:R_0805_HandSoldering, F.Cu at (170.2, 63.5)
- added R17: 6k8, Resistors_SMD:R_0805_HandSoldering, F.Cu at (180.3, 59.1)
- added R18: 6k5, Resistors_SMD:R_0805_HandSoldering, F.Cu at (160.0, 68.6)
- added R19: 6k5, Resistors_SMD:R_0805_HandSoldering, F.Cu at (171.4, 69.8)
- added R2: 1K, Resistors_SMD:R_0805_HandSoldering, F.Cu at (181.6, 71.1)
- added R20: 0, Resistors_SMD:R_0805_HandSoldering, F.Cu at (165.1, 68.6)
- added R21: 0, Resistors_SMD:R_0805_HandSoldering, F.Cu at (176.5, 69.8)
- added R22: 0, Resistors_SMD:R_0805_HandSoldering, F.Cu at (161.3, 61.0)
- added R23: 0, Resistors_SMD:R_0805_HandSoldering, F.Cu at (166.4, 61.0)
- added R24: OC, Resistors_SMD:R_0805_HandSoldering, F.Cu at (171.4, 67.3)
- added R25: OC, Resistors_SMD:R_0805_HandSoldering, F.Cu at (154.9, 66.0)
- added R26: 56, Resistors_SMD:R_0805_HandSoldering, F.Cu at (171.4, 61.0)
- added R27: 4k7, Resistors_SMD:R_0805_HandSoldering, F.Cu at (165.1, 63.5)
- added R28: 4k7, Resistors_SMD:R_0805_HandSoldering, F.Cu at (167.6, 58.4)
- added R3: 1K, Resistors_SMD:R_0805_HandSoldering, F.Cu at (165.1, 71.1)
- added R4: 1k8, Resistors_SMD:R_0805_HandSoldering, F.Cu at (186.7, 68.6)
- added R5: 1K, Resistors_SMD:R_0805_HandSoldering, F.Cu at (160.0, 73.7)
- added R6: 1K, Resistors_SMD:R_0805_HandSoldering, F.Cu at (160.0, 77.5)
- added R7: 6k8, Resistors_SMD:R_0805_HandSoldering, F.Cu at (165.1, 77.5)
- added R8: 6k8, Resistors_SMD:R_0805_HandSoldering, F.Cu at (177.8, 77.5)
- added R9: 0, Resistors_SMD:R_0805_HandSoldering, F.Cu at (154.9, 71.1)
- added RV1: 4k7, Resistors_SMD:R_0805_HandSoldering, F.Cu at (176.5, 67.3)
- added RV2: 4k7, Resistors_SMD:R_0805_HandSoldering, F.Cu at (154.9, 63.5)
- added U1: TRF3701, Housings_VQFN:VQFN-16_3x3mm, F.Cu at (156.8, 59.7)
- added U2: MMZ09332BT1, Resistors_SMD:R_0805_HandSoldering, F.Cu at (181.6, 61.0)
- added U4: Orange Pi zero, orangepi-zero:orangepi-zero, F.Cu at (148.5, 105.0)
- added U5: MCP3421A0T-E/CH, TO_SOT_Packages_SMD:SOT-23-6_Handsoldering, F.Cu at (176.5, 63.5)
- added U6: PCF8563, Housing_SO8:SO-8, F.Cu at (171.4, 76.2)
- added Y1: 32.768Khz, Crystals:Crystal_SMD_G8-2pin_3.2x1.5mm_HandSoldering, F.Cu at (181.6, 67.3)
