File: vhf_uhf_IQ_Modulator_V2.kicad_pcb (KiCad board)
At the start: 2 copper layers, 70 parts, among them J1 Conn_01x06, J2 TEST_1P, J3 Audio-Jack-3, J4 CONN_01X04, J5 SMA Edge FM, Q1 BC817-40, Q2 BC817-40, Q3 BC817-40, U1 TRF3701, U2 MMZ09332BT1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

Commit message: Placing components
Parts:
- added U3: Si570, Oscillators:Oscillator_SMD_SI570_SI571_HandSoldering, F.Cu at (172.7, 82.5)
- J1: value Conn_01x06 -> CONN_01X03; footprint Connectors_Molex:Molex_KK-6410-06_06x2.54mm_Straight -> Pin_Headers:Pin_Header_Straight_1x03_Pitch2.54mm
- J2: footprint Inductors_SMD:L_0805_HandSoldering -> Pin_Headers:Pin_Header_Straight_1x01_Pitch2.54mm
- J3: footprint Connectors_Molex:Molex_KK-6410-03_03x2.54mm_Straight -> Pin_Headers:Pin_Header_Straight_1x03_Pitch2.54mm
- J4: footprint Connectors_Molex:Molex_KK-6410-04_04x2.54mm_Straight -> Pin_Headers:Pin_Header_Straight_1x04_Pitch2.54mm
- RV1, RV2: footprint Resistors_SMD:R_0805_HandSoldering -> Potentiometer_SMD:Potentiometer_Bourns_3314G_Vertical
- U2: footprint Resistors_SMD:R_0805_HandSoldering -> QFN-12-1EP_3x3mm:QFN-12-1EP_3x3mm_P0.5mm_EP1.65x1.65mm
- moved U2 101.7 mm to (231.1, 45.7)
- moved R1 98.2 mm to (234.9, 58.4), turned to 90 degrees
- moved C7 95.4 mm to (243.8, 101.6)
- moved R16 91.3 mm to (221.0, 49.5), turned to 180 degrees
- moved L9 88.3 mm to (232.4, 77.5)
- moved C9 87.8 mm to (236.2, 101.6)
- moved L7 87.6 mm to (232.4, 80.0)
- moved L6 86.9 mm to (232.4, 82.5)
- moved L3 86.2 mm to (232.4, 85.1)
- moved U5 86.0 mm to (210.8, 45.7)
- moved R10 85.7 mm to (223.5, 63.5)
- moved C30 85.7 mm to (232.4, 87.6)
- moved C28 84.8 mm to (232.4, 92.7)
- moved R15 84.4 mm to (219.7, 59.7)
- moved L4 82.8 mm to (231.1, 110.5)
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Connections:
- net /INT renamed Net-(U4-Pad126)
- net /PA01 renamed PA01
- net /PA07 renamed PA07
- C21 pad 2: /PDet -> PDet
- J1 pad 1: Net-(J1-Pad1) -> +5V
- J1 pad 2: Net-(J1-Pad2) -> +3V3
- J1 pad 3: Net-(J1-Pad3) -> GND
- U4 pad 3: Net-(J1-Pad4) -> Net-(U4-Pad3)
- U4 pad 4: Net-(J1-Pad3) -> Net-(U4-Pad4)
- U4 pad 5: Net-(J1-Pad2) -> Net-(U4-Pad5)
- U4 pad 6: Net-(J1-Pad1) -> Net-(U4-Pad6)
- U5 pad 1: /PDet -> PDet
Other:
- rule pad_to_mask_clearance: 0 -> 0.2
