File: vhf_uhf_IQ_Modulator_V2.kicad_pcb (KiCad board)
At the start: 2 copper layers, 71 parts, among them J1 CONN_01X03, J2 TEST_1P, J3 Audio-Jack-3, J4 CONN_01X04, J5 SMA Edge FM, Q1 BC817-40, Q2 BC817-40, Q3 BC817-40, U1 TRF3701, U2 MMZ09332BT1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

Commit message: Placed all components
Parts:
- moved C7 48.3 mm to (156.2, 72.4)
- moved C13 47.1 mm to (158.8, 78.1), turned to 90 degrees
- moved C12 44.6 mm to (165.7, 66.0), turned to 270 degrees
- moved C24 33.5 mm to (172.7, 66.0), turned to 270 degrees
- moved C28 26.1 mm to (179.7, 90.8), turned to 90 degrees
- moved R7 19.1 mm to (179.1, 85.7), turned to 270 degrees
- moved R14 17.9 mm to (182.2, 71.1), turned to 90 degrees
- moved C27 11.4 mm to (187.3, 90.8), turned to 270 degrees
- moved R15 0.63 mm to (183.5, 91.4)
