File: vhf_uhf_IQ_Modulator_V3.kicad_pcb (KiCad board)
At the start: 2 copper layers, 72 parts, among them J1 CONN_01X03, J2 TEST_1P, J3 Audio-Jack-3, J4 CONN_01X04, J5 SMA Edge FM, Q1 BC817-40, Q2 BC817-40, Q3 BC817-40, U1 TRF3701, U2 MMZ09332BT1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

Commit message: added gerber files
Routing:
- net GND: track 316.2 -> 372.8 mm, vias 13 -> 33
- net (no net): track 0.00 -> 12.1 mm, vias 0 -> 8
Changed lines of the file:
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@@
     (thickness 1.6)
     (drawings 8)
-    (tracks 578)
+    (tracks 638)
     (zones 0)
     (modules 72)
@@
     (visible_elements FFFEFFFF)
     (pcbplotparams
-      (layerselection 0x00030_80000001)
-      (usegerberextensions false)
+      (layerselection 0x010f0_80000001)
+      (usegerberextensions true)
       (excludeedgelayer true)
       (linewidth 0.100000)
@@
       (outputformat 1)
       (mirror false)
-      (drillshape 1)
+      (drillshape 0)
       (scaleselection 1)
-      (outputdirectory ""))
+      (outputdirectory Component_position__file))
   )
   (net 0 "")
@@
     (effects (font (size 1.4 1.4) (thickness 0.3)))
   )
+  (via (at 178.943 73.406) (size 0.6) (drill 0.4) (layers F.Cu B.Cu) (net 0))
+  (via (at 178.943 75.057) (size 0.6) (drill 0.4) (layers F.Cu B.Cu) (net 0))
+  (segment (start 178.943 73.406) (end 178.943 75.057) (width 0.3) (layer F.Cu) (net 0))
+  (via (at 166.878 77.597) (size 0.6) (drill 0.4) (layers F.Cu B.Cu) (net 0))
+  (via (at 168.783 77.597) (size 0.6) (drill 0.4) (layers F.Cu B.Cu) (net 0))
+  (segment (start 166.878 77.597) (end 168.783 77.597) (width 0.3) (layer F.Cu) (net 0))
+  (via (at 157.099 86.741) (size 0.6) (drill 0.4) (layers F.Cu B.Cu) (net 0))
+  (via (at 165.608 86.868) (size 0.6) (drill 0.4) (layers F.Cu B.Cu) (net 0))
+  (segment (start 165.608 86.868) (end 163.703 86.868) (width 0.3) (layer F.Cu) (net 0))
+  (via (at 163.703 86.868) (size 0.6) (drill 0.4) (layers F.Cu B.Cu) (net 0))
+  (segment (start 160.274 86.868) (end 163.703 86.868) (width 0.3) (layer B.Cu) (net 0))
+  (segment (start 160.147 86.741) (end 160.274 86.868) (width 0.3) (layer B.Cu) (net 0))
+  (via (at 160.147 86.741) (size 0.6) (drill 0.4) (layers F.Cu B.Cu) (net 0))
+  (segment (start 160.147 86.741) (end 157.099 86.741) (width 0.3) (layer F.Cu) (net 0))
   (via (at 180.467 81.534) (size 0.6) (drill 0.4) (layers F.Cu B.Cu) (net 1))
   (segment (start 180.467 81.534) (end 181.229 82.296) (width 0.25) (layer F.Cu) (net 1))
@@
   (segment (start 182.836 61.221) (end 182.836 64.646) (width 0.25) (layer F.Cu) (net 1))
   (segment (start 182.836 64.646) (end 182.88 64.69) (width 0.25) (layer F.Cu) (net 1))
+  (segment (start 171.704 68.326) (end 172.339 68.326) (width 0.3) (layer B.Cu) (net 2))
+  (segment (start 172.466 69.977) (end 172.466 70.104) (width 0.3) (layer F.Cu) (net 2))
+  (via (at 172.466 69.977) (size 0.6) (drill 0.4) (layers F.Cu B.Cu) (net 2))
+  (segment (start 172.466 68.453) (end 172.466 69.977) (width 0.3) (layer B.Cu) (net 2))
+  (segment (start 172.339 68.326) (end 172.466 68.453) (width 0.3) (layer B.Cu) (net 2))
+  (via (at 162.433 90.551) (size 0.6) (drill 0.4) (layers F.Cu B.Cu) (net 2))
+  (via (at 158.877 90.424) (size 0.6) (drill 0.4) (layers F.Cu B.Cu) (net 2))
+  (segment (start 158.877 90.424) (end 157.353 90.424) (width 0.3) (layer F.Cu) (net 2))
+  (via (at 157.353 90.424) (size 0.6) (drill 0.4) (layers F.Cu B.Cu) (net 2))
+  (segment (start 157.353 93.853) (end 157.353 90.424) (width 0.3) (layer B.Cu) (net 2))
+  (via (at 157.353 93.853) (size 0.6) (drill 0.4) (layers F.Cu B.Cu) (net 2))
+  (segment (start 160.401 93.853) (end 157.353 93.853) (width 0.3) (layer F.Cu) (net 2))
+  (via (at 160.401 93.853) (size 0.6) (drill 0.4) (layers F.Cu B.Cu) (net 2))
+  (segment (start 162.433 93.853) (end 160.401 93.853) (width 0.3) (layer B.Cu) (net 2))
+  (via (at 162.433 93.853) (size 0.6) (drill 0.4) (layers F.Cu B.Cu) (net 2))
+  (segment (start 165.227 93.853) (end 162.433 93.853) (width 0.3) (layer F.Cu) (net 2))
+  (via (at 165.227 93.853) (size 0.6) (drill 0.4) (layers F.Cu B.Cu) (net 2))
+  (segment (start 168.021 93.853) (end 165.227 93.853) (width 0.3) (layer B.Cu) (net 2))
+  (via (at 168.021 93.853) (size 0.6) (drill 0.4) (layers F.Cu B.Cu) (net 2))
+  (segment (start 170.434 93.853) (end 168.021 93.853) (width 0.3) (layer F.Cu) (net 2))
+  (segment (start 170.561 93.726) (end 170.434 93.853) (width 0.3) (layer F.Cu) (net 2))
+  (via (at 170.561 93.726) (size 0.6) (drill 0.4) (layers F.Cu B.Cu) (net 2))
+  (segment (start 170.561 90.551) (end 170.561 93.726) (width 0.3) (layer B.Cu) (net 2))
+  (via (at 170.561 90.551) (size 0.6) (drill 0.4) (layers F.Cu B.Cu) (net 2))
+  (segment (start 168.021 90.551) (end 170.561 90.551) (width 0.3) (layer F.Cu) (net 2))
+  (via (at 168.021 90.551) (size 0.6) (drill 0.4) (layers F.Cu B.Cu) (net 2))
+  (segment (start 165.1 90.551) (end 168.021 90.551) (width 0.3) (layer B.Cu) (net 2))
+  (via (at 165.1 90.551) (size 0.6) (drill 0.4) (layers F.Cu B.Cu) (net 2))
+  (segment (start 165.1 90.551) (end 162.433 90.551) (width 0.3) (layer F.Cu) (net 2))
+  (segment (start 171.45 98.405) (end 169.311 98.405) (width 0.3) (layer F.Cu) (net 2))
+  (via (at 153.162 92.202) (size 0.6) (drill 0.4) (layers F.Cu B.Cu) (net 2))
+  (segment (start 153.162 95.25) (end 153.162 92.202) (width 0.3) (layer F.Cu) (net 2))
+  (via (at 153.162 95.25) (size 0.6) (drill 0.4) (layers F.Cu B.Cu) (net 2))
+  (segment (start 153.162 98.425) (end 153.162 95.25) (width 0.3) (layer B.Cu) (net 2))
+  (via (at 153.162 98.425) (size 0.6) (drill 0.4) (layers F.Cu B.Cu) (net 2))
+  (segment (start 157.861 98.425) (end 153.162 98.425) (width 0.3) (layer F.Cu) (net 2))
+  (via (at 157.861 98.425) (size 0.6) (drill 0.4) (layers F.Cu B.Cu) (net 2))
+  (segment (start 160.528 98.425) (end 157.861 98.425) (width 0.3) (layer B.Cu) (net 2))
+  (segment (start 160.7185 98.2345) (end 160.528 98.425) (width 0.3) (layer B.Cu) (net 2))
+  (via (at 160.7185 98.2345) (size 0.6) (drill 0.4) (layers F.Cu B.Cu) (net 2))
+  (segment (start 165.5445 98.2345) (end 160.7185 98.2345) (width 0.3) (layer F.Cu) (net 2))
+  (segment (start 165.735 98.425) (end 165.5445 98.2345) (width 0.3) (layer F.Cu) (net 2))
+  (via (at 165.735 98.425) (size 0.6) (drill 0.4) (layers F.Cu B.Cu) (net 2))
+  (segment (start 169.291 98.425) (end 165.735 98.425) (width 0.3) (layer B.Cu) (net 2))
+  (segment (start 169.311 98.405) (end 169.291 98.425) (width 0.3) (layer B.Cu) (net 2))
+  (via (at 169.311 98.405) (size 0.6) (drill 0.4) (layers F.Cu B.Cu) (net 2))
   (segment (start 183.45 102.05) (end 183.45 98.61) (width 0.3) (layer B.Cu) (net 2))
   (segment (start 174.69 102.05) (end 183.45 102.05) (width 0.3) (layer B.Cu) (net 2))
