File: _autosave-vhf_uhf_IQ_Modulator_V4.kicad_pcb (KiCad board)
At the start: 2 copper layers, 72 parts, among them J1 CONN_01X03, J2 TEST_1P, J3 Audio-Jack-3, J4 CONN_01X04, J5 SMA Edge FM, Q1 BC817-40, Q2 BC817-40, Q3 BC817-40, U1 TRF3701, U2 MMZ09332BT1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

Commit message: V4 Board Compleat with Gerber
Routing:
- net GND: track 456.4 -> 459.1 mm, vias 71 -> 72
Changed lines of the file:
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@@
     (thickness 1.6)
     (drawings 8)
-    (tracks 768)
+    (tracks 771)
     (zones 0)
     (modules 72)
@@
       (drillshape 0)
       (scaleselection 1)
-      (outputdirectory Component_position__file))
+      (outputdirectory IQ_Modulator_gerber_files/))
   )
   (net 0 "")
@@
   (segment (start 182.836 61.221) (end 182.836 64.646) (width 0.25) (layer F.Cu) (net 1))
   (segment (start 182.836 64.646) (end 182.88 64.69) (width 0.25) (layer F.Cu) (net 1))
-  (segment (start 187.325 73.66) (end 187.325 71.9455) (width 0.3) (layer B.Cu) (net 2) (status 400000))
+  (segment (start 168.148 83.038) (end 168.148 84.5185) (width 0.3) (layer F.Cu) (net 2))
+  (via (at 169.3545 84.5185) (size 0.6) (drill 0.4) (layers F.Cu B.Cu) (net 2))
+  (segment (start 168.148 84.5185) (end 169.3545 84.5185) (width 0.3) (layer F.Cu) (net 2))
+  (segment (start 187.325 73.66) (end 187.325 71.9455) (width 0.3) (layer B.Cu) (net 2))
   (via (at 185.4835 75.311) (size 0.6) (drill 0.4) (layers F.Cu B.Cu) (net 2))
   (segment (start 185.4835 73.152) (end 185.4835 75.311) (width 0.3) (layer B.Cu) (net 2))
@@
   (segment (start 187.325 71.9455) (end 185.4835 71.9455) (width 0.3) (layer F.Cu) (net 2))
   (via (at 187.325 71.9455) (size 0.6) (drill 0.4) (layers F.Cu B.Cu) (net 2))
-  (segment (start 176.53 69.945) (end 176.53 68.6435) (width 0.3) (layer F.Cu) (net 2) (status 400000))
+  (segment (start 176.53 69.945) (end 176.53 68.6435) (width 0.3) (layer F.Cu) (net 2))
   (via (at 176.53 68.6435) (size 0.6) (drill 0.4) (layers F.Cu B.Cu) (net 2))
   (segment (start 181.041 69.993) (end 181.041 71.435) (width 0.3) (layer F.Cu) (net 2))
