File: vhf_uhf_IQ_Modulator_V4.kicad_pcb (KiCad board)
At the start: 2 copper layers, 72 parts, among them J1 CONN_01X03, J2 TEST_1P, J3 Audio-Jack-3, J4 CONN_01X04, J5 SMA Edge FM, Q1 BC817-40, Q2 BC817-40, Q3 BC817-40, U1 TRF3701, U2 MMZ09332BT1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

Commit message: V4 Board Compleat with Gerber
Connections:
- U1 pad 15: Net-(RV2-Pad2) -> Net-(RV1-Pad2)
- U1 pad 16: Net-(RV1-Pad2) -> Net-(RV2-Pad2)
- U2 pad 13: (no net) -> GND
- U2 pad 4: Net-(U2-Pad4) -> (no net)
- U2 pad 5: Net-(U2-Pad5) -> (no net)
- U3 pad 1: Net-(U3-Pad1) -> (no net)
- U4 pad 10: Net-(U4-Pad10) -> (no net)
- U4 pad 108: Net-(U4-Pad108) -> (no net)
- U4 pad 110: Net-(U4-Pad110) -> (no net)
- U4 pad 113: Net-(U4-Pad113) -> (no net)
- U4 pad 115: Net-(U4-Pad115) -> (no net)
- U4 pad 119: Net-(U4-Pad119) -> (no net)
- U4 pad 121: Net-(U4-Pad121) -> (no net)
- U4 pad 122: Net-(U4-Pad122) -> (no net)
- U4 pad 123: Net-(U4-Pad123) -> (no net)
- U4 pad 124: Net-(U4-Pad124) -> (no net)
- U4 pad 126: Net-(U4-Pad126) -> (no net)
- U4 pad 13: Net-(U4-Pad13) -> (no net)
- U4 pad 202: Net-(U4-Pad202) -> (no net)
- U4 pad 203: Net-(U4-Pad203) -> (no net)
- U4 pad 3: Net-(U4-Pad3) -> (no net)
- U4 pad 4: Net-(U4-Pad4) -> (no net)
- U4 pad 5: Net-(U4-Pad5) -> (no net)
- U4 pad 6: Net-(U4-Pad6) -> (no net)
- U4 pad 9: Net-(U4-Pad9) -> (no net)
Routing:
- net GND: track 370.3 -> 459.1 mm, vias 31 -> 72
- net (no net): track 12.1 -> 0.00 mm, vias 8 -> 0
- net Net-(RV2-Pad2): track 16.7 -> 9.74 mm, vias 4 -> 0
- net SDA: track 48.4 -> 53.5 mm
- net Net-(C24-Pad2): track 5.58 -> 7.38 mm
- net Net-(C12-Pad1): track 9.08 -> 7.68 mm, vias 0 -> 2
- net Net-(C7-Pad1): track 18.1 -> 19.2 mm, vias 0 -> 2
- net Net-(RV1-Pad2): track 17.7 -> 16.6 mm, vias 2 -> 0
- net +3V3: track 84.5 -> 85.5 mm
- net +5V: track 177.6 -> 178.4 mm, vias 12 -> 14
- net Net-(Q2-Pad1): track 5.81 -> 6.52 mm
- net Net-(Q3-Pad3): track 16.7 -> 16.1 mm
Other:
- board text added: "SDR_IQ_TX_O_PI"
- board text added: "V1.4"
- board text removed: "SDRTX_O_PI_1"
- board text removed: "V1.0"
