File: vhf_uhf_IQ_Modulator_V4.sch (KiCad schematic (older format))
At the start: 72 parts, among them J1 CONN_01X03, J2 TEST_1P, J3 Audio-Jack-3, J4 CONN_01X04, J5 SMA Edge FM, Q1 BC817-40, Q2 BC817-40, Q3 BC817-40, U1 TRF3701, U2 MMZ09332BT1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

Commit message: V4 Board Compleat with Gerber
Parts:
- U1: footprint TRF3701_new_Anton:VQFN-16_3x3mm -> trf3701_17_pin:VQFN-16_3x3mm_trf3701_new
Connections:
- wire segments 217 -> 220
Other:
- moved on the sheet: C3, RV2
